File: hardware/kicad/inputs-07-08.kicad_sch (KiCad schematic)
At the start: 20 parts, among them J7 PJ-313 5JCJ, J8 PJ-313 5JCJ, U4 TLV9064IDR

Commit message: Clean KiCad 9 root-hierarchy ERC in the generator; add outline DRC to kicad_check
- make_design.py: place symbols, wires, labels and no-connects on the 1.27 mm grid
  (endpoint_off_grid 872 -> 0); add PWR_FLAG on +5V_FUSED and GND, which are fed
  only from off-board USB through passive Pico socket contacts and fuse F1
  (power_pin_not_driven 2 -> 0); generate 74HC4067 Y/Z as passive analog-switch
  terminals instead of bidirectional.
- kicad_check.py: every remaining ERC item needs a reason, endpoint_off_grid and
  lib_symbol_* must be 0, outline-board DRC error count recorded and gated.
- validate.py: exclude '#' power/flag symbols from the physical instance inventory.

Refs #11

Co-Authored-By: Claude Opus 5.5 <noreply@anthropic.com>
Claude-Session: https://claude.ai/code/session_018oLpisCWqu84U1dDpzLDZ4
Other:
- moved on the sheet: C4, C701, C702, C801, C802, D7, D8, J7, J8, R701, R702, R703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
