File: hardware/kicad/inputs-09-10.kicad_sch (KiCad schematic)
At the start: 20 parts, among them J10 PJ-313 5JCJ, J9 PJ-313 5JCJ, U5 TLV9064IDR

Commit message: Clean KiCad 9 root-hierarchy ERC in the generator; add outline DRC to kicad_check
- make_design.py: place symbols, wires, labels and no-connects on the 1.27 mm grid
  (endpoint_off_grid 872 -> 0); add PWR_FLAG on +5V_FUSED and GND, which are fed
  only from off-board USB through passive Pico socket contacts and fuse F1
  (power_pin_not_driven 2 -> 0); generate 74HC4067 Y/Z as passive analog-switch
  terminals instead of bidirectional.
- kicad_check.py: every remaining ERC item needs a reason, endpoint_off_grid and
  lib_symbol_* must be 0, outline-board DRC error count recorded and gated.
- validate.py: exclude '#' power/flag symbols from the physical instance inventory.

Refs #11

Co-Authored-By: Claude Opus 5.5 <noreply@anthropic.com>
Claude-Session: https://claude.ai/code/session_018oLpisCWqu84U1dDpzLDZ4
Other:
- moved on the sheet: C1001, C1002, C5, C901, C902, D10, D9, J10, J9, R1001, R1002, R1003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
