File: hardware/kicad/controls-left.kicad_sch (KiCad schematic)
At the start: 32 parts, among them SW1 SS14MDP2, SW2 SS14MDP2, SW3 SS14MDP2, SW4 SS14MDP2, SW5 SS14MDP2

Commit message: Clean KiCad 9 root-hierarchy ERC in the generator; add outline DRC to kicad_check
- make_design.py: place symbols, wires, labels and no-connects on the 1.27 mm grid
  (endpoint_off_grid 872 -> 0); add PWR_FLAG on +5V_FUSED and GND, which are fed
  only from off-board USB through passive Pico socket contacts and fuse F1
  (power_pin_not_driven 2 -> 0); generate 74HC4067 Y/Z as passive analog-switch
  terminals instead of bidirectional.
- kicad_check.py: every remaining ERC item needs a reason, endpoint_off_grid and
  lib_symbol_* must be 0, outline-board DRC error count recorded and gated.
- validate.py: exclude '#' power/flag symbols from the physical instance inventory.

Refs #11

Co-Authored-By: Claude Opus 5.5 <noreply@anthropic.com>
Claude-Session: https://claude.ai/code/session_018oLpisCWqu84U1dDpzLDZ4
Other:
- moved on the sheet: C1111, C1112, C1121, C1122, C1131, C1132, C1141, C1142, C1151, C1152, R1111, R1112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

Commit message: Generator integrator: apply G01/G02/G08 evidence deltas, candidate footprints (#13)
Applies the cited deltas from #3 (g01-delta.json), #6 (g02-delta.json) and #9
(g08-delta.json) to scripts/make_design.py and catalog/*.json, the only topic
allowed to touch those files.

- G01: record the display-header notes and the R16/R88 backlight default-on
  conflict as a pending_g01_changes proposal only; J30/J31 nets are unchanged,
  per the G01 header-net rule. Documented in the power narrative source too.
- G02: apply the NKK range-switch numeric terminal map (C->3, M->2 vendor
  facts; L->1/H->4 marked OPEN pending panel orientation) and add the
  resolved mechanical facts/open-questions for range, jack, button, display,
  pico-h, socket20 and header20.
- G08: add mpn/jlc_code (with citation, listing_not_allocation) for every
  specification-only candidate that had a source URL and checked date; skip
  r249k/socket20/header20, which have no located citation.
- Fix scripts/fetch_sources.py to download into the gitignored
  reference/downloads/ and write its local fetch log there instead of the
  tracked reference/downloaded/ and reports/source-fetch-local.json.
- Regenerate KiCad sheets/netlist/BOM/MDX/offline HTML; write
  design/evidence/INTEGRATION.md with the footprint-coverage summary and the
  applied/skipped delta table.

validate.py 72/72, kicad_check.py (ERC 0 unexplained, DRC 0, parity PASS,
224/134, 0 differences), test_firmware.py and analyze.py all pass, matching
the pre-existing baseline exactly. G01/G02/G08 stay OPEN.

Co-Authored-By: Claude Sonnet 5 <noreply@anthropic.com>
Claude-Session: https://claude.ai/code/session_018oLpisCWqu84U1dDpzLDZ4
Connections:
- net +3V3A: now also SW1.4 (THROW_RIGHT), SW2.4 (THROW_RIGHT), SW3.4 (THROW_RIGHT), SW4.4 (THROW_RIGHT), SW5.4 (THROW_RIGHT); no longer SW1.H (HIGH_RANGE_LOGICAL), SW2.H (HIGH_RANGE_LOGICAL), SW3.H (HIGH_RANGE_LOGICAL), SW4.H (HIGH_RANGE_LOGICAL), SW5.H (HIGH_RANGE_LOGICAL)
- net CH01_RANGE_W: now also SW1.3 (COMMON); no longer SW1.C (COMMON_LOGICAL)
- net CH02_RANGE_W: now also SW2.3 (COMMON); no longer SW2.C (COMMON_LOGICAL)
- net CH03_RANGE_W: now also SW3.3 (COMMON); no longer SW3.C (COMMON_LOGICAL)
- net CH04_RANGE_W: now also SW4.3 (COMMON); no longer SW4.C (COMMON_LOGICAL)
- net CH05_RANGE_W: now also SW5.3 (COMMON); no longer SW5.C (COMMON_LOGICAL)
- net GND: now also SW1.1 (THROW_LEFT), SW2.1 (THROW_LEFT), SW3.1 (THROW_LEFT), SW4.1 (THROW_LEFT), SW5.1 (THROW_LEFT); no longer SW1.L (LOW_RANGE_LOGICAL), SW2.L (LOW_RANGE_LOGICAL), SW3.L (LOW_RANGE_LOGICAL), SW4.L (LOW_RANGE_LOGICAL), SW5.L (LOW_RANGE_LOGICAL)
- net RANGE_MID: now also SW1.2 (THROW_CENTER), SW2.2 (THROW_CENTER), SW3.2 (THROW_CENTER), SW4.2 (THROW_CENTER), SW5.2 (THROW_CENTER); no longer SW1.M (MID_RANGE_LOGICAL), SW2.M (MID_RANGE_LOGICAL), SW3.M (MID_RANGE_LOGICAL), SW4.M (MID_RANGE_LOGICAL), SW5.M (MID_RANGE_LOGICAL)
