File: hardware/kicad/controls-right.kicad_sch (KiCad schematic)
At the start: 36 parts, among them SW10 SS14MDP2, SW11 TS-1088-AR02016, SW12 TS-1088-AR02016, SW6 SS14MDP2, SW7 SS14MDP2, SW8 SS14MDP2, SW9 SS14MDP2

Commit message: Clean KiCad 9 root-hierarchy ERC in the generator; add outline DRC to kicad_check
- make_design.py: place symbols, wires, labels and no-connects on the 1.27 mm grid
  (endpoint_off_grid 872 -> 0); add PWR_FLAG on +5V_FUSED and GND, which are fed
  only from off-board USB through passive Pico socket contacts and fuse F1
  (power_pin_not_driven 2 -> 0); generate 74HC4067 Y/Z as passive analog-switch
  terminals instead of bidirectional.
- kicad_check.py: every remaining ERC item needs a reason, endpoint_off_grid and
  lib_symbol_* must be 0, outline-board DRC error count recorded and gated.
- validate.py: exclude '#' power/flag symbols from the physical instance inventory.

Refs #11

Co-Authored-By: Claude Opus 5.5 <noreply@anthropic.com>
Claude-Session: https://claude.ai/code/session_018oLpisCWqu84U1dDpzLDZ4
Other:
- moved on the sheet: C1161, C1162, C1171, C1172, C1181, C1182, C1191, C1192, C1201, C1202, C51, C52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

Commit message: Generator integrator: apply G01/G02/G08 evidence deltas, candidate footprints (#13)
Applies the cited deltas from #3 (g01-delta.json), #6 (g02-delta.json) and #9
(g08-delta.json) to scripts/make_design.py and catalog/*.json, the only topic
allowed to touch those files.

- G01: record the display-header notes and the R16/R88 backlight default-on
  conflict as a pending_g01_changes proposal only; J30/J31 nets are unchanged,
  per the G01 header-net rule. Documented in the power narrative source too.
- G02: apply the NKK range-switch numeric terminal map (C->3, M->2 vendor
  facts; L->1/H->4 marked OPEN pending panel orientation) and add the
  resolved mechanical facts/open-questions for range, jack, button, display,
  pico-h, socket20 and header20.
- G08: add mpn/jlc_code (with citation, listing_not_allocation) for every
  specification-only candidate that had a source URL and checked date; skip
  r249k/socket20/header20, which have no located citation.
- Fix scripts/fetch_sources.py to download into the gitignored
  reference/downloads/ and write its local fetch log there instead of the
  tracked reference/downloaded/ and reports/source-fetch-local.json.
- Regenerate KiCad sheets/netlist/BOM/MDX/offline HTML; write
  design/evidence/INTEGRATION.md with the footprint-coverage summary and the
  applied/skipped delta table.

validate.py 72/72, kicad_check.py (ERC 0 unexplained, DRC 0, parity PASS,
224/134, 0 differences), test_firmware.py and analyze.py all pass, matching
the pre-existing baseline exactly. G01/G02/G08 stay OPEN.

Co-Authored-By: Claude Sonnet 5 <noreply@anthropic.com>
Claude-Session: https://claude.ai/code/session_018oLpisCWqu84U1dDpzLDZ4
Connections:
- net +3V3A: now also SW10.4 (THROW_RIGHT), SW6.4 (THROW_RIGHT), SW7.4 (THROW_RIGHT), SW8.4 (THROW_RIGHT), SW9.4 (THROW_RIGHT); no longer SW10.H (HIGH_RANGE_LOGICAL), SW6.H (HIGH_RANGE_LOGICAL), SW7.H (HIGH_RANGE_LOGICAL), SW8.H (HIGH_RANGE_LOGICAL), SW9.H (HIGH_RANGE_LOGICAL)
- net CH06_RANGE_W: now also SW6.3 (COMMON); no longer SW6.C (COMMON_LOGICAL)
- net CH07_RANGE_W: now also SW7.3 (COMMON); no longer SW7.C (COMMON_LOGICAL)
- net CH08_RANGE_W: now also SW8.3 (COMMON); no longer SW8.C (COMMON_LOGICAL)
- net CH09_RANGE_W: now also SW9.3 (COMMON); no longer SW9.C (COMMON_LOGICAL)
- net CH10_RANGE_W: now also SW10.3 (COMMON); no longer SW10.C (COMMON_LOGICAL)
- net GND: now also SW10.1 (THROW_LEFT), SW6.1 (THROW_LEFT), SW7.1 (THROW_LEFT), SW8.1 (THROW_LEFT), SW9.1 (THROW_LEFT); no longer SW10.L (LOW_RANGE_LOGICAL), SW6.L (LOW_RANGE_LOGICAL), SW7.L (LOW_RANGE_LOGICAL), SW8.L (LOW_RANGE_LOGICAL), SW9.L (LOW_RANGE_LOGICAL)
- net RANGE_MID: now also SW10.2 (THROW_CENTER), SW6.2 (THROW_CENTER), SW7.2 (THROW_CENTER), SW8.2 (THROW_CENTER), SW9.2 (THROW_CENTER); no longer SW10.M (MID_RANGE_LOGICAL), SW6.M (MID_RANGE_LOGICAL), SW7.M (MID_RANGE_LOGICAL), SW8.M (MID_RANGE_LOGICAL), SW9.M (MID_RANGE_LOGICAL)
